File: rc-640k.kicad_pcb (KiCad board)
At the start: 2 copper layers, 99.1 x 49.9 mm, 12 parts, among them J1 RC2014, U1 SST39SF040, U2 AS6C1008, U3 74HCT688, U4 74HCT174, U5 74HCT32

Commit message: Move to v1.0
Neaten up board, improve ground plane
Routing:
- net +5V: track 177.9 -> 190.1 mm
- net ~RD: track 65.3 -> 74.1 mm, vias 3 -> 0
- net ~WR: track 106.1 -> 102.2 mm, vias 4 -> 3
- net ~RESET: track 20.9 -> 17.3 mm, vias 0 -> 1
- net /~CFG_CS: track 41.3 -> 39.8 mm
- net ~MREQ: track 78.8 -> 78.0 mm, vias 3 -> 2
Other:
- board text added: "128K+512K RAM/ROM Card"
- board text added: "128K+512K RAM/ROM Card PD108 v1.0"
- board text removed: "128K/512K RAM/ROM Card"
- board text removed: "128K/512K RAM/ROM Card PD108 v1.0"

Commit message: Tweak routing
Routing:
- net MEM_A15: track 83.3 -> 69.7 mm
- net D1: track 56.3 -> 55.2 mm
- net GND: track 39.3 -> 40.2 mm
- net MEM_A16: track 91.4 -> 90.6 mm
- net D0: track 55.7 -> 55.0 mm
- net ~ROM_CS: track 79.2 -> 79.8 mm
- net ~MREQ: track 78.0 -> 78.5 mm
